Commit message: Add hopper training directly from bitbucket.

File: src/legged_robot_description/urdf/monoped.urdf.xacro (robot description, xacro)
@@ -1,3 +1,46 @@
-<robot name="monoped">
+<?xml version="1.0"?>
+<robot xmlns:xacro="http://ros.org/wiki/xacro" name="monoped">
+    <xacro:macro name="monoped_sensors" params="name">
+      <gazebo>
+        <plugin name="p3d_base_controller" filename="libgazebo_ros_p3d.so">
+          <alwaysOn>true</alwaysOn>
+          <updateRate>50.0</updateRate>
+          <bodyName>base</bodyName>
+          <topicName>odom</topicName>
+          <gaussianNoise>0.01</gaussianNoise>
+          <frameName>world</frameName>
+          <xyzOffsets>0 0 0</xyzOffsets>
+          <rpyOffsets>0 0 0</rpyOffsets>
+        </plugin>
+      </gazebo>
+      <!-- Contact Sensor -->
+      <gazebo reference="lowerleg_contactsensor_link">
+        <sensor name="lowerleg_contactsensor_sensor" type="contact">
+          <alwaysOn>true</alwaysOn>
+          <updateRate>30.0</updateRate>
+          <contact>
+            <collision>lowerleg_contactsensor_link_collision_1</collision>
+          </contact>
+          <plugin name="bumper_plugin" filename="libgazebo_ros_bumper.so">
+            <bumperTopicName>lowerleg_contactsensor_state</bumperTopicName>
+            <frameName>lowerleg_contactsensor_link</frameName>
+          </plugin>
+        </sensor>
+      </gazebo>
+      <!-- IMU Sensor -->
+      <gazebo>
+          <plugin name="gazebo_ros_imu_controller" filename="libgazebo_ros_imu.so">
+            <robotNamespace>/${name}</robotNamespace>
+            <topicName>imu/data</topicName>
+            <serviceName>imu/service</serviceName>
+            <bodyName>base</bodyName>
+            <gaussianNoise>0</gaussianNoise>
+            <rpyOffsets>0 0 0</rpyOffsets>
+            <!--<updateRate>50.0</updateRate>-->
+            <alwaysOn>true</alwaysOn>
+          </plugin>
+      </gazebo>
+    </xacro:macro>
+    <xacro:monoped_sensors name="monoped" />
     <gazebo>
       <plugin name="gazebo_ros_control" filename="libgazebo_ros_control.so">
@@ -31,5 +74,5 @@
         <mu1>0.5</mu1>
         <mu2>0.5</mu2>
-        <material>Gazebo/Red</material>
+        <material>Gazebo/Purple</material>
     </gazebo>
     <link name="hipassembly">
@@ -58,5 +101,5 @@
         <mu1>0.5</mu1>
         <mu2>0.5</mu2>
-        <material>Gazebo/Blue</material>
+        <material>Gazebo/Gray</material>
     </gazebo>
     <link name="upperleg">
@@ -85,5 +128,5 @@
         <mu1>0.5</mu1>
         <mu2>0.5</mu2>
-        <material>Gazebo/Blue</material>
+        <material>Gazebo/Green</material>
     </gazebo>
     <link name="lowerleg">
@@ -171,8 +214,8 @@
       <type>transmission_interface/SimpleTransmission</type>
       <joint name="haa_joint">
-        <hardwareInterface>EffortJointInterface</hardwareInterface>
+        <hardwareInterface>hardware_interface/EffortJointInterface</hardwareInterface>
       </joint>
       <actuator name="haa_joint_motor">
-        <hardwareInterface>EffortJointInterface</hardwareInterface>
+        <hardwareInterface>hardware_interface/EffortJointInterface</hardwareInterface>
         <mechanicalReduction>1</mechanicalReduction>
       </actuator>
@@ -181,8 +224,8 @@
       <type>transmission_interface/SimpleTransmission</type>
       <joint name="hfe_joint">
-        <hardwareInterface>EffortJointInterface</hardwareInterface>
+        <hardwareInterface>hardware_interface/EffortJointInterface</hardwareInterface>
       </joint>
       <actuator name="hfe_joint_motor">
-        <hardwareInterface>EffortJointInterface</hardwareInterface>
+        <hardwareInterface>hardware_interface/EffortJointInterface</hardwareInterface>
         <mechanicalReduction>1</mechanicalReduction>
       </actuator>
@@ -191,8 +234,8 @@
       <type>transmission_interface/SimpleTransmission</type>
       <joint name="kfe_joint">
-        <hardwareInterface>EffortJointInterface</hardwareInterface>
+        <hardwareInterface>hardware_interface/EffortJointInterface</hardwareInterface>
       </joint>
       <actuator name="kfe_joint_motor">
-        <hardwareInterface>EffortJointInterface</hardwareInterface>
+        <hardwareInterface>hardware_interface/EffortJointInterface</hardwareInterface>
         <mechanicalReduction>1</mechanicalReduction>
       </actuator>
